Commit message: update 3f top-level xacro to new UR & robotiq repos

File: urdf/ur10e_3f-gripper.xacro (robot description, xacro)
@@ -1,8 +1,10 @@
 <?xml version="1.0"?>
 <robot xmlns:xacro="http://wiki.ros.org/xacro" name="ur10e_3f-gripper">
-  <!-- Import main macro for UR(10e) & Robotiq 3f -->
+  <!-- Import main macro for UR & Robotiq 3f. -->
   <xacro:include filename="$(find ur_gazebo)/urdf/ur_macro.xacro"/>
-  <xacro:include filename="$(find robotiq_3f_gripper_visualization)/cfg/robotiq-3f-gripper_articulated_macro_transmissions.xacro" />
-  <!--Declare arguments -->
+  <xacro:include filename="$(find robotiq_gazebo)/urdf/inc/robotiq_3f_macro.xacro"/>
+  <!-- Declare global arguments. -->
+  <xacro:arg name="prefix" default=""/>
+  <!-- Declare UR arguments. -->
   <xacro:arg name="ur_joint_limit_params" default="(find ur_description)/config/ur10e/joint_limits.yaml"/>
   <xacro:arg name="ur_kinematics_params" default="(find ur_description)/config/ur10e/default_kinematics.yaml"/>
@@ -17,14 +19,24 @@
           controller .yaml files in the 'config' directory.
   -->
-  <xacro:arg name="ur_transmission_hw_interface" default="hardware_interface/EffortJointInterface"/>
+  <xacro:arg name="ur_transmission_hw_interface" default="hardware_interface/PositionJointInterface"/>
   <xacro:arg name="ur_safety_limits" default="false"/>
   <xacro:arg name="ur_safety_pos_margin" default="0.15"/>
   <xacro:arg name="ur_safety_k_position" default="20"/>
-  <xacro:property name="flange_hand">
-    <origin xyz="0.0 0.0 0.045" rpy="${pi/2} 0.0 0.0"/>
-  </xacro:property>
-  <!-- Instantiate the UR(10e) robot and pass it all the required arguments. -->
+  <!-- Declare Robotiq arguments. -->
+  <xacro:arg name="robotiq_joint_limit_params" default="$(find robotiq_3f_description)/config/joint_limits.yaml"/>
+  <xacro:arg name="robotiq_physical_params" default="$(find robotiq_3f_description)/config/physical_parameters.yaml"/>
+  <xacro:arg name="robotiq_visual_params" default="$(find robotiq_3f_description)/config/visual_parameters.yaml"/>
+  <!--
+    legal values:
+      - hardware_interface/PositionJointInterface
+      - hardware_interface/VelocityJointInterface
+      - hardware_interface/EffortJointInterface
+    NOTE: this value must correspond to the controller configured in the
+          controller .yaml files in the 'config' directory.
+  -->
+  <xacro:arg name="robotiq_transmission_hw_interface" default="hardware_interface/EffortJointInterface"/>
+  <!-- Instantiate the UR robot and pass it all the required arguments. -->
   <xacro:ur_robot_gazebo
-    prefix=""
+    prefix="$(arg prefix)"
     joint_limits_parameters_file="$(arg ur_joint_limit_params)"
     kinematics_parameters_file="$(arg ur_kinematics_params)"
@@ -36,5 +48,5 @@
     safety_k_position="$(arg ur_safety_k_position)"
   />
-  <!-- Load the Gazebo standard parameter "world" and fix the base of the UR(10e). -->
+  <!-- Load the Gazebo standard parameter "world" and fix the base of the UR. -->
   <link name="world"/>
   <joint name="world_joint" type="fixed">
@@ -43,12 +55,27 @@
     <origin xyz="0.0 0.0 0.0" rpy="0.0 0.0 0.0"/>
   </joint>
-  <xacro:robotiq-3f-gripper_articulated prefix="" parent="tool0">
-      <xacro:insert_block name="flange_hand"/>
-  </xacro:robotiq-3f-gripper_articulated>
-    <gazebo>
-        <plugin name="ros_control" filename="libgazebo_ros_control.so">
-        <!--robotNamespace>/</robotNamespace-->
-        <!--robotSimType>gazebo_ros_control/DefaultRobotHWSim</robotSimType-->
-        </plugin>
-    </gazebo>
+  <!-- Instantiate the Robotiq 3f and pass it all the required arguments. -->
+  <xacro:robotiq_3f_gazebo
+    prefix="$(arg prefix)"
+    joint_limits_parameters_file="$(arg robotiq_joint_limit_params)"
+    physical_parameters_file="$(arg robotiq_physical_params)"
+    visual_parameters_file="$(arg robotiq_visual_params)"
+    transmission_hw_interface="$(arg robotiq_transmission_hw_interface)"
+  />
+  <!-- Create a fixed joint to mount the Robotiq end effector to the UR. -->
+  <joint name="flange" type="fixed">
+    <parent link="tool0"/>
+    <child link="palm"/>
+    <origin xyz="0.0 0.0 0.045" rpy="${pi/2} 0.0 0.0"/>
+  </joint>
+  <!--
+    Inject Gazebo ROS Control plugin, which allows us to use ros_control
+    controllers to control the virtual robot hw.
+  -->
+  <gazebo>
+      <plugin name="ros_control" filename="libgazebo_ros_control.so">
+      <!--robotNamespace>/</robotNamespace-->
+      <!--robotSimType>gazebo_ros_control/DefaultRobotHWSim</robotSimType-->
+      </plugin>
+  </gazebo>
 </robot>
